Commit message: Remove invalid material definitions

File: robotiq_description/urdf/robotiq_140_gripper.urdf.xacro (robot description, xacro)
@@ -151,7 +151,4 @@
           <box size="0.025 0.06 0.0075"/>
         </geometry>
-        <material name="">
-          <color rgba="0.9 0.0 0.0 1" />
-        </material>
       </collision>
     </link>

File: robotiq_description/urdf/robotiq_85_gripper.urdf.xacro (robot description, xacro)
@@ -124,7 +124,4 @@
            <box size="0.022 0.00635 0.0375"/>
         </geometry>
-        <material name="">
-          <color rgba="0.9 0.0 0.0 1" />
-        </material>
       </collision>
     </link>
