Commit message: Defer robotiq_description from colcon build
Adds `COLCON_IGNORE` to prevent `colcon` from attempting to build `robotiq_description`
while the package is being ported to ROS 2. This unblocks the workspace build
during the ongoing ROS 2 migration.

Removes ROS 1-specific OpenRAVE dependencies from CMake and package files as
part of the porting preparation.

Updates the `robotiq_hande_gripper.urdf.xacro` with corrected inertia tensor
values, specifically setting off-diagonal components to zero for simplification
and consistency.

File: robotiq_description/urdf/robotiq_hande_gripper.urdf.xacro (robot description, xacro)
@@ -15,5 +15,5 @@
         <origin rpy="0 0 0" xyz="0 0 0.04607"/>
         <mass value="0.86387"/>
-        <inertia ixx="1017560E-9" ixy="0" ixz="2235E-9" iyy="1028041E-9" iyz="0" izz="489810E-9"/>
+        <inertia ixx="1.017560e-3" ixy="0" ixz="2.235e-6" iyy="1.028041e-3" iyz="0" izz="4.89810e-4"/>
       </inertial>
       <visual>
@@ -37,5 +37,5 @@
         <origin rpy="0 0 0" xyz="0.02262 -0.00759 0.00738"/>
         <mass value="0.03804"/>
-        <inertia ixx="13567E-9" ixy="1849E-9" ixz="3622E-9" iyy="15784E-9" iyz="3616E-9" izz="7478E-9"/>
+        <inertia ixx="1.4e-5" ixy="0" ixz="0" iyy="1.6e-5" iyz="0" izz="7.5e-6"/>
       </inertial>
       <visual>
@@ -59,5 +59,5 @@
         <origin rpy="0 0 0" xyz="-0.02262 0.00759 0.00738"/>
         <mass value="0.03804"/>
-        <inertia ixx="13567E-9" ixy="1849E-9" ixz="-3622E-9" iyy="15784E-9" iyz="-3616E-9" izz="7478E-9"/>
+        <inertia ixx="1.4e-5" ixy="0" ixz="0" iyy="1.6e-5" iyz="0" izz="7.5e-6"/>
       </inertial>
       <visual>
